Commit message: feat(nav.gps): Add GPS link

File: src/openmower/description/robot.urdf.xacro (robot description, xacro)
@@ -6,4 +6,5 @@
     <xacro:property name="robot" value="${xacro.load_yaml(robot_yaml)}"/>
     <xacro:include filename="robot_core.xacro" />
+    <xacro:include filename="gps.xacro" />
     <xacro:if value="$(arg use_ros2_control)">
         <xacro:include filename="ros2_control.xacro" />

File: src/openmower/description/robot_core.xacro (robot description, xacro)
@@ -19,5 +19,5 @@
     <xacro:property name="caster_wheel_offset_x" value="${robot['caster_wheel']['offset'][0]}"/>
     <xacro:property name="caster_wheel_offset_y" value="${robot['caster_wheel']['offset'][1]}"/>
-    <xacro:property name="caster_wheel_offset_z" value="${wheel_offset_z - wheel_radius + caster_wheel_radius}"/>
+    <xacro:property name="caster_wheel_offset_z" value="${wheel_offset_z - wheel_radius + caster_wheel_radius*2}"/>
     <material name="white">
         <color rgba="1 1 1 1" />
