Commit message: robot localization

File: src/openmower/description/gazebo_control.xacro (robot description, xacro)
@@ -21,9 +21,9 @@
       <state_interface name="velocity"/>
     </joint>
-    <joint name="mower_joint">
+    <!-- <joint name="mower_joint">
       <command_interface name="effort">
       </command_interface>
       <state_interface name="effort"/>
-    </joint>
+    </joint> -->
   </ros2_control>
   <gazebo>

File: src/openmower/description/robot_core.xacro (robot description, xacro)
@@ -126,5 +126,5 @@
     </gazebo>
     <!-- MOWER LINK -->
-    <joint name="mower_joint" type="continuous">
+    <!-- <joint name="mower_joint" type="continuous">
         <parent link="base_link"/>
         <child link="mower"/>
@@ -150,5 +150,5 @@
     <gazebo reference="mower">
         <material>Gazebo/Red</material>
-    </gazebo>
+    </gazebo> -->
     <!-- LEFT CASTER WHEEL LINK -->
     <joint name="left_caster_wheel_joint" type="fixed">
