Commit message: Adjust robot URDF values

File: src/openmower/description/gps.xacro (robot description, xacro)
@@ -4,23 +4,10 @@
         <parent link="base_link"/>
         <child link="gps"/>
-        <origin xyz="0.3 0 0.05" rpy="0 0 0"/>
+        <origin xyz="${robot['gps']['antenna']['offset'][0]} ${robot['gps']['antenna']['offset'][1]} ${robot['gps']['antenna']['offset'][2]}" rpy="0 0 0"/>
     </joint>
     <link name="gps">
-        <collision>
-            <origin xyz="0 0 0" rpy="0 0 0"/>
-            <geometry>
-                <box size="0.08 0.08 0.04"></box>
-            </geometry>
-        </collision>
-        <visual>
-            <origin xyz="0 0 0" rpy="0 0 0"/>
-            <geometry>
-                <box size="0.08 0.08 0.04"></box>
-            </geometry>
-            <material name="black"/>
-        </visual>
         <sensor name="navsat_sensor" type="navsat">
           <always_on>1</always_on>
-          <update_rate>30</update_rate>
+          <update_rate>5</update_rate>
           <topic>gps</topic>
         </sensor>

File: src/openmower/description/imu.xacro (robot description, xacro)
@@ -4,20 +4,7 @@
         <parent link="base_link"/>
         <child link="imu"/>
-        <origin xyz="0.5 0 0.05" rpy="0 0 0"/>
+        <origin xyz="${robot['imu']['chip']['offset'][0]} ${robot['imu']['chip']['offset'][1]} ${robot['imu']['chip']['offset'][2]}" rpy="0 0 0"/>
     </joint>
     <link name="imu">
-        <collision>
-            <origin xyz="0 0 0" rpy="0 0 0"/>
-            <geometry>
-                <box size="0.08 0.08 0.04"></box>
-            </geometry>
-        </collision>
-        <visual>
-            <origin xyz="0 0 0" rpy="0 0 0"/>
-            <geometry>
-                <box size="0.08 0.08 0.04"></box>
-            </geometry>
-            <material name="red"/>
-        </visual>
     </link>
     <gazebo reference="imu">

File: src/openmower/description/robot.urdf.xacro (robot description, xacro)
@@ -8,5 +8,5 @@
     <xacro:include filename="gps.xacro" />
     <xacro:include filename="imu.xacro" />
-    <xacro:include filename="camera.xacro" />
+<!--    <xacro:include filename="camera.xacro" />-->
     <xacro:if value="$(arg use_ros2_control)">
         <xacro:include filename="ros2_control.xacro" />

File: src/openmower/description/robot_core.xacro (robot description, xacro)
@@ -15,9 +15,9 @@
     <xacro:property name="wheel_offset_y" value="${robot['wheel']['offset'][1]}"/>
     <xacro:property name="wheel_offset_z" value="${robot['wheel']['offset'][2]}"/>
-    <xacro:property name="caster_wheel_radius" value="${robot['caster_wheel']['mass']}"/>
+    <xacro:property name="caster_wheel_radius" value="${robot['caster_wheel']['radius']}"/>
     <xacro:property name="caster_wheel_mass" value="${robot['caster_wheel']['mass']}"/>
     <xacro:property name="caster_wheel_offset_x" value="${robot['caster_wheel']['offset'][0]}"/>
     <xacro:property name="caster_wheel_offset_y" value="${robot['caster_wheel']['offset'][1]}"/>
-    <xacro:property name="caster_wheel_offset_z" value="${wheel_offset_z - wheel_radius + caster_wheel_radius*2}"/>
+    <xacro:property name="caster_wheel_offset_z" value="${wheel_offset_z - wheel_radius + caster_wheel_radius}"/>
     <material name="white">
         <color rgba="1 1 1 1" />
@@ -159,5 +159,5 @@
     <!-- LEFT CASTER WHEEL LINK -->
     <joint name="left_caster_wheel_joint" type="fixed">
-        <parent link="chassis"/>
+        <parent link="base_link"/>
         <child link="left_caster_wheel"/>
         <origin xyz="${caster_wheel_offset_x} ${caster_wheel_offset_y} ${caster_wheel_offset_z}"/>
@@ -168,5 +168,5 @@
                 <sphere radius="${caster_wheel_radius}"/>
             </geometry>
-            <material name="white"/>
+            <material name="black"/>
         </visual>
         <collision>
@@ -180,5 +180,5 @@
     </link>
     <gazebo reference="left_caster_wheel">
-        <material>Gazebo/White</material>
+        <material>Gazebo/Black</material>
         <mu1 value="0.001"/>
         <mu2 value="0.001"/>
@@ -186,5 +186,5 @@
     <!-- RIGHT CASTER WHEEL LINK -->
     <joint name="right_caster_wheel_joint" type="fixed">
-        <parent link="chassis"/>
+        <parent link="base_link"/>
         <child link="right_caster_wheel"/>
         <origin xyz="${caster_wheel_offset_x} ${-caster_wheel_offset_y} ${caster_wheel_offset_z}"/>
@@ -195,5 +195,5 @@
                 <sphere radius="${caster_wheel_radius}"/>
             </geometry>
-            <material name="white"/>
+            <material name="black"/>
         </visual>
         <collision>
@@ -207,5 +207,5 @@
     </link>
     <gazebo reference="right_caster_wheel">
-        <material>Gazebo/White</material>
+        <material>Gazebo/Black</material>
         <mu1 value="0.001"/>
         <mu2 value="0.001"/>
