Commit message: map server services

File: description/gazebo_control.xacro (robot description, xacro)
@@ -30,5 +30,5 @@
     <!-- Joint state publisher -->
     <plugin filename="gz_ros2_control-system" name="gz_ros2_control::GazeboSimROS2ControlPlugin">
-      <parameters>$(find openmower)/config/controllers.yaml</parameters>
+      <parameters>$(find open_mower_next)/config/controllers.yaml</parameters>
     </plugin>
   </gazebo>

File: description/robot.urdf.xacro (robot description, xacro)
@@ -3,5 +3,5 @@
     <xacro:arg name="use_ros2_control" default="true"/>
     <xacro:arg name="sim_mode" default="false"/>
-    <xacro:property name="robot_yaml" value="$(find openmower)/config/hardware/yardforce500.yaml" />
+    <xacro:property name="robot_yaml" value="$(find open_mower_next)/config/hardware/yardforce500.yaml" />
     <xacro:property name="robot" value="${xacro.load_yaml(robot_yaml)}"/>
     <xacro:include filename="robot_core.xacro" />

Commit message: make sim great again

File: description/gazebo_control.xacro (robot description, xacro)
@@ -21,9 +21,11 @@
       <state_interface name="velocity"/>
     </joint>
-    <!-- <joint name="mower_joint">
+    <joint name="mower_joint">
       <command_interface name="effort">
       </command_interface>
+      <state_interface name="position"/>
+      <state_interface name="velocity"/>
       <state_interface name="effort"/>
-    </joint> -->
+    </joint>
   </ros2_control>
   <gazebo>
@@ -34,4 +36,31 @@
       <robot_param_node>robot_state_publisher</robot_param_node>
     </plugin>
+    <!-- Physics settings -->
+    <physics type="ode">
+      <max_step_size>0.001</max_step_size>
+      <real_time_factor>1.0</real_time_factor>
+      <real_time_update_rate>1000</real_time_update_rate>
+      <ode>
+        <solver>
+          <type>quick</type>
+          <iters>50</iters>
+          <sor>1.3</sor>
+        </solver>
+        <constraints>
+          <cfm>0.0</cfm>
+          <erp>0.2</erp>
+          <contact_max_correcting_vel>100.0</contact_max_correcting_vel>
+          <contact_surface_layer>0.001</contact_surface_layer>
+        </constraints>
+      </ode>
+      <magnetic_field>6.0e-6 2.3e-5 -4.2e-5</magnetic_field>
+      <atmosphere type='adiabatic'/>
+      <wind/>
+    </physics>
+    <!-- Add damping to the model -->
+    <velocity_decay>
+      <linear>0.1</linear>
+      <angular>0.1</angular>
+    </velocity_decay>
   </gazebo>
 </robot>

File: description/robot_core.xacro (robot description, xacro)
@@ -85,4 +85,5 @@
         <origin xyz="${wheel_offset_x} ${wheel_offset_y} ${wheel_offset_z}" rpy="-${pi/2} 0 0" />
         <axis xyz="0 0 1"/>
+        <dynamics damping="0.1" friction="0.2"/>
     </joint>
     <link name="left_wheel">
@@ -95,5 +96,5 @@
         <collision>
             <geometry>
-                <sphere radius="${wheel_radius}"/>
+                <cylinder radius="${wheel_radius}" length="${wheel_thickness}"/>
             </geometry>
         </collision>
@@ -104,4 +105,13 @@
     <gazebo reference="left_wheel">
         <material>Gazebo/Blue</material>
+        <mu1 value="1.0"/>
+        <mu2 value="1.0"/>
+        <kp value="10000000.0" />
+        <kd value="1.0" />
+        <fdir1 value="1 0 0"/>
+        <minDepth>0.005</minDepth>
+        <maxVel>1.0</maxVel>
+        <slip1>0.0</slip1>
+        <slip2>0.0</slip2>
     </gazebo>
     <!-- RIGHT WHEEL LINK -->
@@ -111,4 +121,5 @@
         <origin xyz="${wheel_offset_x} ${-wheel_offset_y} ${wheel_offset_z}" rpy="${pi/2} 0 0" />
         <axis xyz="0 0 -1"/>
+        <dynamics damping="0.1" friction="0.2"/>
     </joint>
     <link name="right_wheel">
@@ -121,5 +132,5 @@
         <collision>
             <geometry>
-                <sphere radius="${wheel_radius}"/>
+                <cylinder radius="${wheel_radius}" length="${wheel_thickness}"/>
             </geometry>
         </collision>
@@ -130,4 +141,13 @@
     <gazebo reference="right_wheel">
         <material>Gazebo/Blue</material>
+        <mu1 value="1.0"/>
+        <mu2 value="1.0"/>
+        <kp value="10000000.0" />
+        <kd value="1.0" />
+        <fdir1 value="1 0 0"/>
+        <minDepth>0.005</minDepth>
+        <maxVel>1.0</maxVel>
+        <slip1>0.0</slip1>
+        <slip2>0.0</slip2>
     </gazebo>
     <!-- MOWER LINK -->
@@ -135,5 +155,5 @@
         <parent link="base_link"/>
         <child link="mower"/>
-        <origin xyz="${robot['mower']['offset'][0]} ${robot['mower']['offset'][1]} ${robot['mower']['offset'][2]}" rpy="${pi/2} 0 0" />
+        <origin xyz="${robot['mower']['offset'][0]} ${robot['mower']['offset'][1]} ${robot['mower']['offset'][2]}" rpy="0 0 0" />
         <axis xyz="0 0 -1"/>
     </joint>
@@ -147,5 +167,5 @@
         <collision>
             <geometry>
-                <sphere radius="${robot['mower']['cut_radius']}"/>
+                <cylinder radius="${robot['mower']['cut_radius']}" length="${robot['mower']['thickness']}"/>
             </geometry>
         </collision>
@@ -156,10 +176,28 @@
     <gazebo reference="mower">
         <material>Gazebo/Red</material>
+        <mu1 value="0.5"/>
+        <mu2 value="0.5"/>
     </gazebo>
     <!-- LEFT CASTER WHEEL LINK -->
-    <joint name="left_caster_wheel_joint" type="fixed">
-        <parent link="base_link"/>
+    <!-- Caster Swivel -->
+    <joint name="left_caster_swivel_joint" type="continuous">
+        <parent link="base_link"/>
+        <child link="left_caster_swivel"/>
+        <origin xyz="${caster_wheel_offset_x} ${caster_wheel_offset_y} ${caster_wheel_offset_z}"/>
+        <axis xyz="0 0 1"/>
+    </joint>
+    <link name="left_caster_swivel">
+        <xacro:inertial_sphere mass="0.01" radius="0.01">
+            <origin xyz="0 0 0" rpy="0 0 0"/>
+        </xacro:inertial_sphere>
+    </link>
+    <gazebo reference="left_caster_swivel">
+        <material>Gazebo/Black</material>
+    </gazebo>
+    <joint name="left_caster_wheel_joint" type="continuous">
+        <parent link="left_caster_swivel"/>
         <child link="left_caster_wheel"/>
-        <origin xyz="${caster_wheel_offset_x} ${caster_wheel_offset_y} ${caster_wheel_offset_z}"/>
+        <origin xyz="0 0 0" rpy="-${pi/2} 0 0"/>
+        <axis xyz="0 0 1"/>
     </joint>
     <link name="left_caster_wheel">
@@ -172,5 +210,5 @@
         <collision>
             <geometry>
-                <sphere radius="${caster_wheel_radius}"/>
+                <sphere radius="${caster_wheel_radius * 0.97}"/>
             </geometry>
         </collision>
@@ -183,10 +221,28 @@
         <mu1 value="0.001"/>
         <mu2 value="0.001"/>
+        <kp value="10000.0" />
+        <kd value="1.0" />
     </gazebo>
     <!-- RIGHT CASTER WHEEL LINK -->
-    <joint name="right_caster_wheel_joint" type="fixed">
-        <parent link="base_link"/>
+    <!-- Caster Swivel -->
+    <joint name="right_caster_swivel_joint" type="continuous">
+        <parent link="base_link"/>
+        <child link="right_caster_swivel"/>
+        <origin xyz="${caster_wheel_offset_x} ${-caster_wheel_offset_y} ${caster_wheel_offset_z}"/>
+        <axis xyz="0 0 1"/>
+    </joint>
+    <link name="right_caster_swivel">
+        <xacro:inertial_sphere mass="0.01" radius="0.01">
+            <origin xyz="0 0 0" rpy="0 0 0"/>
+        </xacro:inertial_sphere>
+    </link>
+    <gazebo reference="right_caster_swivel">
+        <material>Gazebo/Black</material>
+    </gazebo>
+    <joint name="right_caster_wheel_joint" type="continuous">
+        <parent link="right_caster_swivel"/>
         <child link="right_caster_wheel"/>
-        <origin xyz="${caster_wheel_offset_x} ${-caster_wheel_offset_y} ${caster_wheel_offset_z}"/>
+        <origin xyz="0 0 0" rpy="-${pi/2} 0 0"/>
+        <axis xyz="0 0 1"/>
     </joint>
     <link name="right_caster_wheel">
@@ -199,5 +255,5 @@
         <collision>
             <geometry>
-                <sphere radius="${caster_wheel_radius}"/>
+                <sphere radius="${caster_wheel_radius * 0.97}"/>
             </geometry>
         </collision>
@@ -210,4 +266,13 @@
         <mu1 value="0.001"/>
         <mu2 value="0.001"/>
+        <kp value="10000.0" />
+        <kd value="1.0" />
+    </gazebo>
+    <!-- Global collision settings -->
+    <gazebo>
+        <self_collide>0</self_collide>
+        <collision_detector>bullet</collision_detector>
+        <static>0</static>
+        <gravity>1</gravity>
     </gazebo>
 </robot>
