Commit message: fix ros2_control

File: description/robot_core.xacro (robot description, xacro)
@@ -1,4 +1,4 @@
 <?xml version="1.0"?>
-<robot xmlns:xacro="http://www.ros.org/wiki/xacro" >
+<robot xmlns:xacro="http://www.ros.org/wiki/xacro">
     <xacro:include filename="inertial_macros.xacro"/>
     <xacro:property name="chassis_length" value="${robot['chassis']['length']}"/>
@@ -39,7 +39,5 @@
     </link>
     <gazebo>
-        <plugin
-                filename="gz-sim-pose-publisher-system"
-                name="gz::sim::systems::PosePublisher">
+        <plugin filename="gz-sim-pose-publisher-system" name="gz::sim::systems::PosePublisher">
             <use_pose_vector_msg>true</use_pose_vector_msg>
             <publish_nested_model_pose>true</publish_nested_model_pose>
@@ -134,5 +132,5 @@
     </gazebo>
     <!-- MOWER LINK -->
-    <!-- <joint name="mower_joint" type="continuous">
+    <joint name="mower_joint" type="continuous">
         <parent link="base_link"/>
         <child link="mower"/>
@@ -158,5 +156,5 @@
     <gazebo reference="mower">
         <material>Gazebo/Red</material>
-    </gazebo> -->
+    </gazebo>
     <!-- LEFT CASTER WHEEL LINK -->
     <joint name="left_caster_wheel_joint" type="fixed">

File: description/ros2_control.xacro (robot description, xacro)
@@ -41,16 +41,15 @@
                 <param name="joint_type">continuous</param>
                 <param name="port">${vesc['serial']['mower']}</param>
-                <param name="command_mode">effort</param>
-                <param name="num_rotor_poles">4</param>
-                <param name="num_hall_sensors">6</param>
-                <param name="gear_ratio">1.0</param>
-                <param name="torque_const">2.0</param>
+                <param name="command_mode">velocity</param>
             </hardware>
             <joint name="mower_joint">
                 <command_interface name="position"/>
-                <command_interface name="velocity"/>
+                <command_interface name="velocity">
+                    <param name="min">-1</param>
+                    <param name="max">1</param>
+                </command_interface>
                 <command_interface name="effort">
-                    <param name="min">-10</param>
-                    <param name="max">10</param>
+                    <param name="min">-1</param>
+                    <param name="max">1</param>
                 </command_interface>
                 <state_interface name="position"/>

Commit message: OpenMowerNext (#27)
* Use depot.dev build

* add setup action

* make docker-entrypoint.sh executable

* fix build

* fix project id

* remove rosdep.yml reference

* this build works

* fix

* fix

* add description

* tune stuff a bit

* dada

* fix

* fix ros2_control

* extend docker-entrypoint.sh

* fix

* things

* run mower_controller

* get things work better

* include nodejs and npm for docs

* make sim great again

* :fire:

* update docs CI

* fix docs ci

* OpenMowerNext

File: description/robot_core.xacro (robot description, xacro)
@@ -1,4 +1,4 @@
 <?xml version="1.0"?>
-<robot xmlns:xacro="http://www.ros.org/wiki/xacro" >
+<robot xmlns:xacro="http://www.ros.org/wiki/xacro">
     <xacro:include filename="inertial_macros.xacro"/>
     <xacro:property name="chassis_length" value="${robot['chassis']['length']}"/>
@@ -39,7 +39,5 @@
     </link>
     <gazebo>
-        <plugin
-                filename="gz-sim-pose-publisher-system"
-                name="gz::sim::systems::PosePublisher">
+        <plugin filename="gz-sim-pose-publisher-system" name="gz::sim::systems::PosePublisher">
             <use_pose_vector_msg>true</use_pose_vector_msg>
             <publish_nested_model_pose>true</publish_nested_model_pose>
@@ -87,4 +85,5 @@
         <origin xyz="${wheel_offset_x} ${wheel_offset_y} ${wheel_offset_z}" rpy="-${pi/2} 0 0" />
         <axis xyz="0 0 1"/>
+        <dynamics damping="0.1" friction="0.2"/>
     </joint>
     <link name="left_wheel">
@@ -97,5 +96,5 @@
         <collision>
             <geometry>
-                <sphere radius="${wheel_radius}"/>
+                <cylinder radius="${wheel_radius}" length="${wheel_thickness}"/>
             </geometry>
         </collision>
@@ -106,4 +105,13 @@
     <gazebo reference="left_wheel">
         <material>Gazebo/Blue</material>
+        <mu1 value="1.0"/>
+        <mu2 value="1.0"/>
+        <kp value="10000000.0" />
+        <kd value="1.0" />
+        <fdir1 value="1 0 0"/>
+        <minDepth>0.005</minDepth>
+        <maxVel>1.0</maxVel>
+        <slip1>0.0</slip1>
+        <slip2>0.0</slip2>
     </gazebo>
     <!-- RIGHT WHEEL LINK -->
@@ -113,4 +121,5 @@
         <origin xyz="${wheel_offset_x} ${-wheel_offset_y} ${wheel_offset_z}" rpy="${pi/2} 0 0" />
         <axis xyz="0 0 -1"/>
+        <dynamics damping="0.1" friction="0.2"/>
     </joint>
     <link name="right_wheel">
@@ -123,5 +132,5 @@
         <collision>
             <geometry>
-                <sphere radius="${wheel_radius}"/>
+                <cylinder radius="${wheel_radius}" length="${wheel_thickness}"/>
             </geometry>
         </collision>
@@ -132,10 +141,19 @@
     <gazebo reference="right_wheel">
         <material>Gazebo/Blue</material>
+        <mu1 value="1.0"/>
+        <mu2 value="1.0"/>
+        <kp value="10000000.0" />
+        <kd value="1.0" />
+        <fdir1 value="1 0 0"/>
+        <minDepth>0.005</minDepth>
+        <maxVel>1.0</maxVel>
+        <slip1>0.0</slip1>
+        <slip2>0.0</slip2>
     </gazebo>
     <!-- MOWER LINK -->
-    <!-- <joint name="mower_joint" type="continuous">
+    <joint name="mower_joint" type="continuous">
         <parent link="base_link"/>
         <child link="mower"/>
-        <origin xyz="${robot['mower']['offset'][0]} ${robot['mower']['offset'][1]} ${robot['mower']['offset'][2]}" rpy="${pi/2} 0 0" />
+        <origin xyz="${robot['mower']['offset'][0]} ${robot['mower']['offset'][1]} ${robot['mower']['offset'][2]}" rpy="0 0 0" />
         <axis xyz="0 0 -1"/>
     </joint>
@@ -149,5 +167,5 @@
         <collision>
             <geometry>
-                <sphere radius="${robot['mower']['cut_radius']}"/>
+                <cylinder radius="${robot['mower']['cut_radius']}" length="${robot['mower']['thickness']}"/>
             </geometry>
         </collision>
@@ -158,10 +176,28 @@
     <gazebo reference="mower">
         <material>Gazebo/Red</material>
-    </gazebo> -->
+        <mu1 value="0.5"/>
+        <mu2 value="0.5"/>
+    </gazebo>
     <!-- LEFT CASTER WHEEL LINK -->
-    <joint name="left_caster_wheel_joint" type="fixed">
-        <parent link="base_link"/>
+    <!-- Caster Swivel -->
+    <joint name="left_caster_swivel_joint" type="continuous">
+        <parent link="base_link"/>
+        <child link="left_caster_swivel"/>
+        <origin xyz="${caster_wheel_offset_x} ${caster_wheel_offset_y} ${caster_wheel_offset_z}"/>
+        <axis xyz="0 0 1"/>
+    </joint>
+    <link name="left_caster_swivel">
+        <xacro:inertial_sphere mass="0.01" radius="0.01">
+            <origin xyz="0 0 0" rpy="0 0 0"/>
+        </xacro:inertial_sphere>
+    </link>
+    <gazebo reference="left_caster_swivel">
+        <material>Gazebo/Black</material>
+    </gazebo>
+    <joint name="left_caster_wheel_joint" type="continuous">
+        <parent link="left_caster_swivel"/>
         <child link="left_caster_wheel"/>
-        <origin xyz="${caster_wheel_offset_x} ${caster_wheel_offset_y} ${caster_wheel_offset_z}"/>
+        <origin xyz="0 0 0" rpy="-${pi/2} 0 0"/>
+        <axis xyz="0 0 1"/>
     </joint>
     <link name="left_caster_wheel">
@@ -174,5 +210,5 @@
         <collision>
             <geometry>
-                <sphere radius="${caster_wheel_radius}"/>
+                <sphere radius="${caster_wheel_radius * 0.97}"/>
             </geometry>
         </collision>
@@ -185,10 +221,28 @@
         <mu1 value="0.001"/>
         <mu2 value="0.001"/>
+        <kp value="10000.0" />
+        <kd value="1.0" />
     </gazebo>
     <!-- RIGHT CASTER WHEEL LINK -->
-    <joint name="right_caster_wheel_joint" type="fixed">
-        <parent link="base_link"/>
+    <!-- Caster Swivel -->
+    <joint name="right_caster_swivel_joint" type="continuous">
+        <parent link="base_link"/>
+        <child link="right_caster_swivel"/>
+        <origin xyz="${caster_wheel_offset_x} ${-caster_wheel_offset_y} ${caster_wheel_offset_z}"/>
+        <axis xyz="0 0 1"/>
+    </joint>
+    <link name="right_caster_swivel">
+        <xacro:inertial_sphere mass="0.01" radius="0.01">
+            <origin xyz="0 0 0" rpy="0 0 0"/>
+        </xacro:inertial_sphere>
+    </link>
+    <gazebo reference="right_caster_swivel">
+        <material>Gazebo/Black</material>
+    </gazebo>
+    <joint name="right_caster_wheel_joint" type="continuous">
+        <parent link="right_caster_swivel"/>
         <child link="right_caster_wheel"/>
-        <origin xyz="${caster_wheel_offset_x} ${-caster_wheel_offset_y} ${caster_wheel_offset_z}"/>
+        <origin xyz="0 0 0" rpy="-${pi/2} 0 0"/>
+        <axis xyz="0 0 1"/>
     </joint>
     <link name="right_caster_wheel">
@@ -201,5 +255,5 @@
         <collision>
             <geometry>
-                <sphere radius="${caster_wheel_radius}"/>
+                <sphere radius="${caster_wheel_radius * 0.97}"/>
             </geometry>
         </collision>
@@ -212,4 +266,13 @@
         <mu1 value="0.001"/>
         <mu2 value="0.001"/>
+        <kp value="10000.0" />
+        <kd value="1.0" />
+    </gazebo>
+    <!-- Global collision settings -->
+    <gazebo>
+        <self_collide>0</self_collide>
+        <collision_detector>bullet</collision_detector>
+        <static>0</static>
+        <gravity>1</gravity>
     </gazebo>
 </robot>

Commit message: make sim charging more reliable

File: description/robot_core.xacro (robot description, xacro)
@@ -35,4 +35,7 @@
         <color rgba="1 0 0 1"/>
     </material>
+    <material name="green">
+        <color rgba="0 0.8 0 1"/>
+    </material>
     <!-- BASE LINK -->
     <link name="base_link">
@@ -78,4 +81,31 @@
     <gazebo reference="chassis">
         <material>Gazebo/Orange</material>
+    </gazebo>
+    <!-- CHARGING PORT LINK -->
+    <xacro:property name="charging_port_radius" value="0.01"/>
+    <xacro:property name="charging_port_mass" value="0.01"/>
+    <joint name="charging_port_joint" type="fixed">
+        <parent link="base_link"/>
+        <child link="charging_port"/>
+        <origin xyz="${chassis_offset_x + chassis_length} ${chassis_offset_y} ${chassis_offset_z + chassis_height/2}" rpy="0 0 0"/>
+    </joint>
+    <link name="charging_port">
+        <visual>
+            <geometry>
+                <sphere radius="${charging_port_radius}"/>
+            </geometry>
+            <material name="green"/>
+        </visual>
+        <collision>
+            <geometry>
+                <sphere radius="${charging_port_radius}"/>
+            </geometry>
+        </collision>
+        <xacro:inertial_sphere mass="${charging_port_mass}" radius="${charging_port_radius}">
+            <origin xyz="0 0 0" rpy="0 0 0"/>
+        </xacro:inertial_sphere>
+    </link>
+    <gazebo reference="charging_port">
+        <material>Gazebo/Green</material>
     </gazebo>
     <!-- LEFT WHEEL LINK -->
